File: Filter+LNA/Eagle_Specific/ADSB_AMP_V3.brd (EAGLE design)
At the start: 105.3 x 47 mm, 12 parts, among them U1 BFP420, X1 SMA-142-0701-801/806, X2 SMA-142-0701-801/806

Commit message: Updated Layout
Parts:
- moved U$1 28.9 mm to (3.17, 3.49), flipped to the bottom, turned to 180 degrees
Routing:
- net GND: track 2.68 -> 20.2 mm
Other:
- board size 105.3 x 47 mm -> 105.3 x 45.7 mm
Changed lines of the file:
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@@
 <plain>
 <wire x1="-85.725" y1="-20.32" x2="19.52625" y2="-20.32" width="0" layer="20"/>
-<wire x1="19.52625" y1="-20.32" x2="19.52625" y2="26.6575" width="0" layer="20"/>
-<wire x1="19.52625" y1="26.6575" x2="-85.725" y2="26.6575" width="0" layer="20"/>
-<wire x1="-85.725" y1="26.6575" x2="-85.725" y2="-20.32" width="0" layer="20"/>
+<wire x1="19.52625" y1="-20.32" x2="19.52625" y2="25.3875" width="0" layer="20"/>
+<wire x1="19.52625" y1="25.3875" x2="-85.725" y2="25.3875" width="0" layer="20"/>
+<wire x1="-85.725" y1="25.3875" x2="-85.725" y2="-20.32" width="0" layer="20"/>
 <polygon width="0.0254" layer="29">
 <vertex x="5.08" y="2.54"/>
@@
 <vertex x="-80.01" y="-16.51"/>
 <vertex x="-77.47" y="-19.05"/>
-<vertex x="-19.3675" y="-19.05"/>
-<vertex x="5.08" y="-3.81"/>
+<vertex x="2.2225" y="-19.05"/>
+<vertex x="5.08" y="-16.51"/>
 <vertex x="5.08" y="5.08"/>
 </polygon>
@@
 <vertex x="-80.01" y="-16.51"/>
 <vertex x="-77.47" y="-19.05"/>
-<vertex x="-19.3675" y="-19.05"/>
-<vertex x="5.08" y="-3.81"/>
+<vertex x="2.2225" y="-19.05"/>
+<vertex x="5.08" y="-16.51"/>
 <vertex x="5.08" y="21.59"/>
 <vertex x="2.54" y="24.13"/>
@@
 <elements>
 <element name="U1" library="transistor-small-signal" package="SOT343_INFINEON" value="BFP420" x="9.8425" y="4.7625" smashed="yes" rot="R315">
-<attribute name="NAME" x="8.151628125" y="4.673228125" size="0.6096" layer="25" rot="R45"/>
+<attribute name="NAME" x="8.469128125" y="5.308228125" size="0.6096" layer="25" rot="R45"/>
 </element>
 <element name="C1" library="Passives" package="0805" value="100pF" x="5.8674" y="4.38785" smashed="yes" rot="R33.7">
-<attribute name="NAME" x="4.9779" y="4.977684375" size="0.6096" layer="25" font="vector" ratio="19" rot="R37.5"/>
+<attribute name="NAME" x="5.6129" y="5.612684375" size="0.6096" layer="25" font="vector" ratio="19" rot="R37.5"/>
 </element>
 <element name="R1" library="Passives" package="0805" value="22K" x="8.255" y="1.27" smashed="yes" rot="R315">
-<attribute name="NAME" x="8.659109375" y="2.257828125" size="0.6096" layer="25" font="vector" ratio="19" rot="R315"/>
+<attribute name="NAME" x="6.754109375" y="0.352828125" size="0.6096" layer="25" font="vector" ratio="19" rot="R315"/>
 </element>
 <element name="X1" library="con-coax" package="J502-ND-142-0701-801/806" value="SMA-142-0701-801/806" x="-85.725" y="2.38125" smashed="yes">
@@
 </element>
 <element name="C2" library="Passives" package="0805" value="100pF" x="12.54125" y="2.54" smashed="yes">
-<attribute name="NAME" x="11.01725" y="3.683" size="0.6096" layer="25" font="vector" ratio="19"/>
+<attribute name="NAME" x="12.28725" y="3.683" size="0.6096" layer="25" font="vector" ratio="19"/>
 </element>
 <element name="TP3" library="Pads_Test_Points" package="SMD_8_8" value="TEST_POINTS8_8" x="-79.21625" y="2.69875" smashed="yes"/>
 <element name="TP4" library="Pads_Test_Points" package="SMD_8_8" value="TEST_POINTS8_8" x="2.69875" y="2.2225" smashed="yes"/>
-<element name="U$1" library="logos" package="RTLSDR-LARGE" value="RTLSDR-LARGE" x="19.05" y="-20.6375" rot="R90"/>
+<element name="U$1" library="logos" package="RTLSDR-LARGE" value="RTLSDR-LARGE" x="3.175" y="3.4925" rot="MR180"/>
 </elements>
 <signals>
@@
 <vertex x="-85.725" y="-20.32"/>
 <vertex x="19.52625" y="-20.32"/>
-<vertex x="19.52625" y="26.67"/>
-<vertex x="-85.725" y="26.67"/>
+<vertex x="19.52625" y="25.4"/>
+<vertex x="-85.725" y="25.4"/>
 </polygon>
 <contactref element="TP2" pad="1"/>
@@
 <wire x1="9.948565625" y1="6.773565625" x2="10.16" y2="6.985" width="0.635" layer="1" curve="-90"/>
 <via x="9.8425" y="2.54" extent="1-16" drill="0.508" diameter="0.762"/>
-<wire x1="-83.1596" y1="-2.03835" x2="-83.1596" y2="-2.03835" width="0" layer="19" extent="1-16"/>
-<wire x1="-83.1596" y1="6.80085" x2="-83.1596" y2="6.80085" width="0" layer="19" extent="1-16"/>
-<wire x1="16.96085" y1="6.80085" x2="16.96085" y2="6.80085" width="0" layer="19" extent="1-16"/>
-<wire x1="16.96085" y1="-2.03835" x2="16.96085" y2="-2.03835" width="0" layer="19" extent="1-16"/>
 <wire x1="9.630365625" y1="3.843259375" x2="9.630365625" y2="2.752134375" width="0.635" layer="1"/>
 <wire x1="9.630365625" y1="2.752134375" x2="9.8425" y2="2.54" width="0.635" layer="1" curve="90"/>
@@
 <via x="-83.185" y="-2.2225" extent="1-16" drill="0.508" diameter="0.762"/>
 <via x="-81.5975" y="-2.2225" extent="1-16" drill="0.508" diameter="0.762"/>
+<wire x1="16.96085" y1="-2.03835" x2="15.74165" y2="-2.03835" width="0.635" layer="1"/>
+<wire x1="15.74165" y1="-2.03835" x2="15.5575" y2="-2.2225" width="0.635" layer="1" curve="90"/>
+<wire x1="15.5575" y1="-2.2225" x2="18.415" y2="-2.2225" width="0.635" layer="1"/>
+<wire x1="16.96085" y1="6.80085" x2="15.69085" y2="6.80085" width="0.635" layer="1"/>
+<wire x1="15.69085" y1="6.80085" x2="15.5575" y2="6.6675" width="0.635" layer="1" curve="90"/>
+<wire x1="15.5575" y1="6.6675" x2="18.7325" y2="6.6675" width="0.635" layer="1"/>
+<wire x1="18.7325" y1="6.6675" x2="17.0942" y2="6.6675" width="0.635" layer="1"/>
+<wire x1="17.0942" y1="6.6675" x2="16.96085" y2="6.80085" width="0.635" layer="1" curve="-90"/>
+<wire x1="-83.1596" y1="-2.03835" x2="-84.58835" y2="-2.03835" width="0.635" layer="1"/>
+<wire x1="-84.58835" y1="-2.03835" x2="-84.7725" y2="-2.2225" width="0.635" layer="1" curve="90"/>
+<wire x1="-84.7725" y1="-2.2225" x2="-84.455" y2="-2.2225" width="0.635" layer="1"/>
+<wire x1="-84.455" y1="-2.2225" x2="-83.34375" y2="-2.2225" width="0.635" layer="1"/>
+<wire x1="-83.34375" y1="-2.2225" x2="-83.1596" y2="-2.03835" width="0.635" layer="1" curve="90"/>
+<wire x1="-83.1596" y1="6.80085" x2="-84.63915" y2="6.80085" width="0.635" layer="1"/>
+<wire x1="-84.63915" y1="6.80085" x2="-84.7725" y2="6.6675" width="0.635" layer="1" curve="90"/>
+<wire x1="-84.7725" y1="6.6675" x2="-83.29295" y2="6.6675" width="0.635" layer="1"/>
+<wire x1="-83.29295" y1="6.6675" x2="-83.1596" y2="6.80085" width="0.635" layer="1" curve="90"/>
 </signal>
 <signal name="N$2">
@@
 </signal>
 </signals>
-<errors>
-</errors>
 </board>
 </drawing>
